Commit message: [ADD] 1. add cnn-vae 2. add cnn debug viz 3. add height_scan_points python scripts

File: source/unitree_rl_lab/unitree_rl_lab/assets/robots/g1_23dof_description/urdf/g1_23dof.urdf (robot description, URDF)
Before this commit: robot g1_23dof_rev_1_0, 36 links, 35 joints
Links:
- removed link left_foot_hook
- removed link left_hand_hook
- removed link right_foot_hook
- removed link right_hand_hook
- added link left_foot_hook0, mass 0.01; visual sphere radius=0.01
- added link left_foot_hook1, mass 0.01; visual sphere radius=0.01
- added link left_foot_hook2, mass 0.01; visual sphere radius=0.01
- added link right_foot_hook0, mass 0.01; visual sphere radius=0.01
- added link right_foot_hook1, mass 0.01; visual sphere radius=0.01
- added link right_foot_hook2, mass 0.01; visual sphere radius=0.01
Joints:
- removed joint left_foot_hook_sphere_fixed
- removed joint left_wrist_roll_rubber_hand_sphere_fixed
- removed joint right_foot_hook_sphere_fixed
- removed joint right_wrist_roll_rubber_hand_sphere_fixed
- added joint left_foot_hook0_sphere_fixed: type fixed, parent left_ankle_pitch_link, child left_foot_hook0, origin xyz=0.035 0. -0.05 rpy=0 0 0
- added joint left_foot_hook1_sphere_fixed: type fixed, parent left_ankle_pitch_link, child left_foot_hook1, origin xyz=0.11 0. -0.05 rpy=0 0 0
- added joint left_foot_hook2_sphere_fixed: type fixed, parent left_ankle_pitch_link, child left_foot_hook2, origin xyz=-0.04 0. -0.05 rpy=0 0 0
- added joint right_foot_hook0_sphere_fixed: type fixed, parent right_ankle_pitch_link, child right_foot_hook0, origin xyz=0.035 0. -0.05 rpy=0 0 0
- added joint right_foot_hook1_sphere_fixed: type fixed, parent right_ankle_pitch_link, child right_foot_hook1, origin xyz=0.11 0. -0.05 rpy=0 0 0
- added joint right_foot_hook2_sphere_fixed: type fixed, parent right_ankle_pitch_link, child right_foot_hook2, origin xyz=-0.04 0. -0.05 rpy=0 0 0

Commit message: [ADD] 1. 添加gas box origin 2. 添加actioin clip 3. 添加阶梯地形 4. 修改gas penalty奖励的判断link

File: source/unitree_rl_lab/unitree_rl_lab/assets/robots/g1_23dof_description/urdf/g1_23dof.urdf (robot description, URDF)
Before this commit: robot g1_23dof_rev_1_0, 38 links, 37 joints
Joints:
- joint left_foot_hook0_sphere_fixed: origin xyz=0.035 0. -0.05 rpy=0 0 0 -> xyz=0.11 0. -0.05 rpy=0 0 0
- joint left_foot_hook1_sphere_fixed: origin xyz=0.11 0. -0.05 rpy=0 0 0 -> xyz=0.035 0. -0.05 rpy=0 0 0
- joint right_foot_hook0_sphere_fixed: origin xyz=0.035 0. -0.05 rpy=0 0 0 -> xyz=0.11 0. -0.05 rpy=0 0 0
- joint right_foot_hook1_sphere_fixed: origin xyz=0.11 0. -0.05 rpy=0 0 0 -> xyz=0.035 0. -0.05 rpy=0 0 0
